Commit message: gazebo

File: omnimate_description/urdf/omnimate.urdf.xacro (robot description, xacro)
@@ -8,4 +8,5 @@
         <inertial>
             <origin xyz="0.00498197982182523 5.70233829969297E-05 -0.0121008098068578" rpy="0 0 0" />
+            <!--<origin xyz="0.00498197982182523 5.70233829969297E-05 -0.0121008098068578" rpy="0 0 0" />-->
             <mass value="0.486218814966626" />
             <inertia
@@ -50,6 +51,5 @@
             <origin xyz="0 0 0" rpy="0 0 0" />
             <geometry>
-                <mesh
-                    filename="package://omnimate_description/meshes/wheels/front_right_wheel_X3.STL" />
+                <sphere radius="0.07162"/>
             </geometry>
         </collision>
@@ -75,6 +75,5 @@
             <origin xyz="0 0 0" rpy="0 0 0" />
             <geometry>
-                <mesh
-                    filename="package://omnimate_description/meshes/wheels/front_left_wheel_X3.STL" />
+                <sphere radius="0.07162"/>
             </geometry>
         </collision>
@@ -102,6 +101,5 @@
             <origin xyz="0 0 0" rpy="0 0 0" />
             <geometry>
-                <mesh
-                    filename="package://omnimate_description/meshes/wheels/back_right_wheel_X3.STL" />
+                <sphere radius="0.07162"/>
             </geometry>
         </collision>
@@ -129,6 +127,5 @@
             <origin xyz="0 0 0" rpy="0 0 0" />
             <geometry>
-                <mesh
-                    filename="package://omnimate_description/meshes/wheels/back_left_wheel_X3.STL" />
+                <sphere radius="0.07162"/>
             </geometry>
         </collision>
