Commit message: Cambios en el description para corregir fallos en el avance del robot

File: Omnimate_ros1/yahboom_new_description/urdf/yahboom.urdf.xacro (robot description, xacro)
@@ -1,23 +1,22 @@
 <?xml version="1.0"?>
-<robot name="yahboomcar"
-    xmlns:xacro="http://www.ros.org/wiki/xacro">
+<robot name="yahboomcar" xmlns:xacro="http://www.ros.org/wiki/xacro">
     <!-- Include files-->
-    <!--<xacro:include filename="$(find yahboom_new_description)/urdf/yahboom_gazebo.xacro"/>-->
-    <!--<xacro:include filename="$(find yahboom_new_description)/urdf/sensors/imu.xacro"/>
-    <xacro:include filename="$(find yahboom_new_description)/urdf/sensors/lidar.xacro"/>-->
-    <xacro:include filename="$(find yahboom_new_description)/urdf/_l515.urdf.xacro" />
-    <!-- Material-->
-    <material name="green">
-        <color rgba="0 1.0 0 1"/>
-    </material>
-    <material name="black">
-        <color rgba="0.0 0.0 0.0 1"/>
-    </material>
-    <material name="purple">
-        <color rgba="0.5 0 0.5 1"/>
-    </material>
-    <!-- Links-->
+    <xacro:include filename="$(find yahboom_new_description)/urdf/common_properties.xacro"/>
+    <xacro:include filename="$(find yahboom_new_description)/urdf/yahboom.gazebo.xacro"/>
+    <!-- Links and joints -->
     <link name="base_footprint"/>
+    <joint name="base_joint" type="fixed">
+        <origin xyz="0 0 0.07" rpy="0 0 0"/>
+        <parent link="base_footprint"/>
+        <child link="base_link"/>
+        <axis xyz="0 0 1"/>
+    </joint>
     <link name="imu_link"/>
+    <joint name="imu_joint" type="fixed">
+        <origin xyz="0 0 0.07" rpy="0 0 0"/>
+        <parent link="base_footprint"/>
+        <child link="imu_link"/>
+        <axis xyz="0 0 1"/>
+    </joint>
     <link name="base_link">
         <inertial>
@@ -60,4 +59,11 @@
         </collision>
     </link>
+    <joint name="front_left_joint" type="continuous">
+        <origin xyz="0.11797 0.084101 -0.0389" rpy="-1.5708 0 0"/>
+        <parent link="base_link"/>
+        <child link="front_left_wheel"/>
+        <axis xyz="0 0 1" rpy="0 0 0"/>
+        <limit effort="100" velocity="1"/>
+    </joint>
     <link name="front_right_wheel">
         <inertial>
@@ -80,4 +86,11 @@
         </collision>
     </link>
+    <joint name="front_right_joint" type="continuous">
+        <origin xyz="0.11797 -0.084099 -0.0389" rpy="1.5708 0 0"/>
+        <parent link="base_link"/>
+        <child link="front_right_wheel"/>
+        <axis xyz="0 0 1" rpy="0 0 0"/>
+        <limit effort="100" velocity="1"/>
+    </joint>
     <link name="back_left_wheel">
         <inertial>
@@ -100,4 +113,11 @@
         </collision>
     </link>
+    <joint name="back_left_joint" type="continuous">
+        <origin xyz="-0.10203 0.084101 -0.0395" rpy="-1.5708 0 0"/>
+        <parent link="base_link"/>
+        <child link="back_left_wheel"/>
+        <axis xyz="0 0 1" rpy="0 0 0"/>
+        <limit effort="100" velocity="1"/>
+    </joint>
     <link name="back_right_wheel">
         <inertial>
@@ -120,4 +140,11 @@
         </collision>
     </link>
+    <joint name="back_right_joint" type="continuous">
+        <origin xyz="-0.10203 -0.084099 -0.0395" rpy="1.5708 0 0"/>
+        <parent link="base_link"/>
+        <child link="back_right_wheel"/>
+        <axis xyz="0 0 1" rpy="0 0 0"/>
+        <limit effort="100" velocity="1"/>
+    </joint>
     <link name="camera_base">
         <inertial>
@@ -140,54 +167,4 @@
         </collision>
     </link>
-    <link name="camera_reference_link"/>
-    <link name="base_scan">
-        <inertial>
-            <origin xyz="0.00070942 0.0008187 0.013068" rpy="0 0 0"/>
-            <mass value="0.045513" />
-            <inertia ixx="8.6093E-06" ixy="1.7259E-07" ixz="6.5083E-09" iyy="8.4939E-06" iyz="5.3304E-08" izz="1.0141E-05"/>
-        </inertial>
-        <visual>
-            <origin xyz="0 0 0" rpy="0 0 0"/>
-            <geometry>
-                <mesh filename="package://yahboom_new_description/meshes/laser_link.STL"/>
-            </geometry>
-            <material name="black"/>
-        </visual>
-        <collision>
-            <origin xyz="0 0 0" rpy="0 0 0"/>
-            <geometry>
-                <mesh filename="package://yahboom_new_description/meshes/laser_link.STL"/>
-            </geometry>
-        </collision>
-    </link>
-    <!-- Joints-->
-    <joint name="front_left_joint" type="continuous">
-        <origin xyz="0.11797 0.084101 -0.0389" rpy="-1.5708 0 0"/>
-        <parent link="base_link"/>
-        <child link="front_left_wheel"/>
-        <axis xyz="0 0 1" rpy="0 0 0"/>
-        <limit effort="100" velocity="1"/>
-    </joint>
-    <joint name="front_right_joint" type="continuous">
-        <origin xyz="0.11797 -0.084099 -0.0389" rpy="1.5708 0 0"/>
-        <parent link="base_link"/>
-        <child link="front_right_wheel"/>
-        <axis xyz="0 0 1" rpy="0 0 0"/>
-        <limit effort="100" velocity="1"/>
-    </joint>
-    <joint name="back_left_joint" type="continuous">
-        <origin xyz="-0.10203 0.084101 -0.0395" rpy="-1.5708 0 0"/>
-        <parent link="base_link"/>
-        <child link="back_left_wheel"/>
-        <axis xyz="0 0 1" rpy="0 0 0"/>
-        <limit effort="100" velocity="1"/>
-    </joint>
-    <joint name="back_right_joint" type="continuous">
-        <origin xyz="-0.10203 -0.084099 -0.0395" rpy="1.5708 0 0"/>
-        <parent link="base_link"/>
-        <child link="back_right_wheel"/>
-        <axis xyz="0 0 1" rpy="0 0 0"/>
-        <limit effort="100" velocity="1"/>
-    </joint>
     <joint name="camera_base_joint" type="fixed">
         <origin xyz="0.14057 0 0.066" rpy="0 0 0"/>
@@ -196,4 +173,5 @@
         <axis xyz="0 0 0"/>
     </joint>
+    <link name="camera_reference_link"/>
     <joint name="camera_reference_joint" type="fixed">
         <!--<origin xyz="-0.020646 -0.0011633 0.088297" rpy="1.5708 0 0"/>-->
@@ -203,20 +181,35 @@
         <axis xyz="0 0 0"/>
     </joint>
+    <joint name="camera_reference_joint" type="fixed">
+        <!--<origin xyz="-0.020646 -0.0011633 0.088297" rpy="1.5708 0 0"/>-->
+        <origin xyz="-0.006 -0.0011633 0.057797" rpy="0 0 0"/>
+        <parent link="camera_base"/>
+        <child link="camera_reference_link"/>
+        <axis xyz="0 0 0"/>
+    </joint>
+    <link name="base_scan">
+        <inertial>
+            <origin xyz="0.00070942 0.0008187 0.013068" rpy="0 0 0"/>
+            <mass value="0.045513" />
+            <inertia ixx="8.6093E-06" ixy="1.7259E-07" ixz="6.5083E-09" iyy="8.4939E-06" iyz="5.3304E-08" izz="1.0141E-05"/>
+        </inertial>
+        <visual>
+            <origin xyz="0 0 0" rpy="0 0 0"/>
+            <geometry>
+                <mesh filename="package://yahboom_new_description/meshes/laser_link.STL"/>
+            </geometry>
+            <material name="black"/>
+        </visual>
+        <collision>
+            <origin xyz="0 0 0" rpy="0 0 0"/>
+            <geometry>
+                <mesh filename="package://yahboom_new_description/meshes/laser_link.STL"/>
+            </geometry>
+        </collision>
+    </link>
     <joint name="laser_joint" type="fixed">
         <origin xyz="0.11596 -0.0019383 0" rpy="0 0 0"/>
         <parent link="base_link"/>
         <child link="base_scan"/>
-        <axis xyz="0 0 1"/>
-    </joint>
-    <joint name="base_joint" type="fixed">
-        <origin xyz="0 0 0.07" rpy="0 0 0"/>
-        <parent link="base_footprint"/>
-        <child link="base_link"/>
-        <axis xyz="0 0 1"/>
-    </joint>
-    <joint name="imu_joint" type="fixed">
-        <origin xyz="0 0 0.07" rpy="0 0 0"/>
-        <parent link="base_footprint"/>
-        <child link="imu_link"/>
         <axis xyz="0 0 1"/>
     </joint>
